Commit message: Improvements

File: Navigation/urdf/ultrabot.urdf.xacro (robot description, xacro)
@@ -22,6 +22,17 @@
   <xacro:property name="base_width" value="0.5" />
   <xacro:property name="base_height" value="0.3" />
-  <xacro:property name="laser_x" value="0.25" />            <!-- LiDAR front offset -->
-  <xacro:property name="laser_z" value="0.20" />            <!-- LiDAR height -->
+  <!-- Sensor mounting positions -->
+  <xacro:property name="lidar_front_x" value="0.25" />      <!-- Front 2D LiDAR -->
+  <xacro:property name="lidar_front_z" value="0.20" />
+  <xacro:property name="lidar_rear_x" value="-0.25" />      <!-- Rear 2D LiDAR -->
+  <xacro:property name="lidar_rear_z" value="0.20" />
+  <xacro:property name="lidar_3d_x" value="0.0" />          <!-- 3D LiDAR (Ouster) top center -->
+  <xacro:property name="lidar_3d_z" value="0.35" />
+  <xacro:property name="realsense_front_left_x" value="0.22" />   <!-- Front-left RealSense D455 -->
+  <xacro:property name="realsense_front_left_y" value="0.15" />
+  <xacro:property name="realsense_front_left_z" value="0.15" />
+  <xacro:property name="realsense_front_right_x" value="0.22" />  <!-- Front-right RealSense D455 -->
+  <xacro:property name="realsense_front_right_y" value="-0.15" />
+  <xacro:property name="realsense_front_right_z" value="0.15" />
   <!-- ===================================================================== -->
   <!-- MATERIALS (Visual Colors for RViz) -->
@@ -146,7 +157,7 @@
   </joint>
   <!-- ===================================================================== -->
-  <!-- LASER FRAME (LiDAR Sensor - Front Center) -->
-  <!-- ===================================================================== -->
-  <link name="laser_frame">
+  <!-- FRONT 2D LIDAR (e.g., SICK TiM571, Hokuyo UST-10LX) -->
+  <!-- ===================================================================== -->
+  <link name="scan_front_link">
     <visual>
       <origin xyz="0 0 0" rpy="0 0 0"/>
@@ -170,9 +181,149 @@
     </inertial>
   </link>
-  <!-- Joint: base_link → laser_frame (fixed, front center position) -->
-  <joint name="laser_joint" type="fixed">
-    <parent link="base_link"/>
+  <joint name="scan_front_joint" type="fixed">
+    <parent link="base_link"/>
+    <child link="scan_front_link"/>
+    <origin xyz="${lidar_front_x} 0 ${lidar_front_z}" rpy="0 0 0"/>
+  </joint>
+  <!-- ===================================================================== -->
+  <!-- REAR 2D LIDAR (Rear Coverage for Obstacle Detection) -->
+  <!-- ===================================================================== -->
+  <link name="scan_rear_link">
+    <visual>
+      <origin xyz="0 0 0" rpy="0 0 0"/>
+      <geometry>
+        <cylinder radius="0.05" length="0.05"/>
+      </geometry>
+      <material name="red"/>
+    </visual>
+    <collision>
+      <origin xyz="0 0 0" rpy="0 0 0"/>
+      <geometry>
+        <cylinder radius="0.05" length="0.05"/>
+      </geometry>
+    </collision>
+    <inertial>
+      <origin xyz="0 0 0" rpy="0 0 0"/>
+      <mass value="0.5"/>
+      <inertia ixx="0.001" ixy="0.0" ixz="0.0"
+               iyy="0.001" iyz="0.0"
+               izz="0.001"/>
+    </inertial>
+  </link>
+  <joint name="scan_rear_joint" type="fixed">
+    <parent link="base_link"/>
+    <child link="scan_rear_link"/>
+    <origin xyz="${lidar_rear_x} 0 ${lidar_rear_z}" rpy="0 0 ${pi}"/>  <!-- 180° rotation -->
+  </joint>
+  <!-- ===================================================================== -->
+  <!-- 3D LIDAR (Ouster OS1-64/OS1-128 - PointCloud2) -->
+  <!-- ===================================================================== -->
+  <link name="ouster_link">
+    <visual>
+      <origin xyz="0 0 0" rpy="0 0 0"/>
+      <geometry>
+        <cylinder radius="0.06" length="0.08"/>
+      </geometry>
+      <material name="black"/>
+    </visual>
+    <collision>
+      <origin xyz="0 0 0" rpy="0 0 0"/>
+      <geometry>
+        <cylinder radius="0.06" length="0.08"/>
+      </geometry>
+    </collision>
+    <inertial>
+      <origin xyz="0 0 0" rpy="0 0 0"/>
+      <mass value="0.8"/>
+      <inertia ixx="0.002" ixy="0.0" ixz="0.0"
+               iyy="0.002" iyz="0.0"
+               izz="0.002"/>
+    </inertial>
+  </link>
+  <joint name="ouster_joint" type="fixed">
+    <parent link="base_link"/>
+    <child link="ouster_link"/>
+    <origin xyz="${lidar_3d_x} 0 ${lidar_3d_z}" rpy="0 0 0"/>
+  </joint>
+  <!-- ===================================================================== -->
+  <!-- REALSENSE D455 - FRONT LEFT -->
+  <!-- ===================================================================== -->
+  <link name="camera_front_left_link">
+    <visual>
+      <origin xyz="0 0 0" rpy="0 0 0"/>
+      <geometry>
+        <box size="0.026 0.090 0.025"/>  <!-- D455 dimensions -->
+      </geometry>
+      <material name="black"/>
+    </visual>
+    <collision>
+      <origin xyz="0 0 0" rpy="0 0 0"/>
+      <geometry>
+        <box size="0.026 0.090 0.025"/>
+      </geometry>
+    </collision>
+    <inertial>
+      <origin xyz="0 0 0" rpy="0 0 0"/>
+      <mass value="0.12"/>  <!-- ~120g -->
+      <inertia ixx="0.0001" ixy="0.0" ixz="0.0"
+               iyy="0.0001" iyz="0.0"
+               izz="0.0001"/>
+    </inertial>
+  </link>
+  <joint name="camera_front_left_joint" type="fixed">
+    <parent link="base_link"/>
+    <child link="camera_front_left_link"/>
+    <origin xyz="${realsense_front_left_x} ${realsense_front_left_y} ${realsense_front_left_z}" rpy="0 0 0"/>
+  </joint>
+  <!-- Optical frame (RealSense convention: Z forward, Y down) -->
+  <link name="camera_front_left_depth_optical_frame"/>
+  <joint name="camera_front_left_depth_optical_joint" type="fixed">
+    <parent link="camera_front_left_link"/>
+    <child link="camera_front_left_depth_optical_frame"/>
+    <origin xyz="0 0 0" rpy="${-pi/2} 0 ${-pi/2}"/>  <!-- Rotate to optical frame -->
+  </joint>
+  <!-- ===================================================================== -->
+  <!-- REALSENSE D455 - FRONT RIGHT -->
+  <!-- ===================================================================== -->
+  <link name="camera_front_right_link">
+    <visual>
+      <origin xyz="0 0 0" rpy="0 0 0"/>
+      <geometry>
+        <box size="0.026 0.090 0.025"/>
+      </geometry>
+      <material name="black"/>
+    </visual>
+    <collision>
+      <origin xyz="0 0 0" rpy="0 0 0"/>
+      <geometry>
+        <box size="0.026 0.090 0.025"/>
+      </geometry>
+    </collision>
+    <inertial>
+      <origin xyz="0 0 0" rpy="0 0 0"/>
+      <mass value="0.12"/>
+      <inertia ixx="0.0001" ixy="0.0" ixz="0.0"
+               iyy="0.0001" iyz="0.0"
+               izz="0.0001"/>
+    </inertial>
+  </link>
+  <joint name="camera_front_right_joint" type="fixed">
+    <parent link="base_link"/>
+    <child link="camera_front_right_link"/>
+    <origin xyz="${realsense_front_right_x} ${realsense_front_right_y} ${realsense_front_right_z}" rpy="0 0 0"/>
+  </joint>
+  <!-- Optical frame -->
+  <link name="camera_front_right_depth_optical_frame"/>
+  <joint name="camera_front_right_depth_optical_joint" type="fixed">
+    <parent link="camera_front_right_link"/>
+    <child link="camera_front_right_depth_optical_frame"/>
+    <origin xyz="0 0 0" rpy="${-pi/2} 0 ${-pi/2}"/>
+  </joint>
+  <!-- Legacy compatibility: keep laser_frame pointing to front 2D LiDAR -->
+  <link name="laser_frame"/>
+  <joint name="laser_frame_joint" type="fixed">
+    <parent link="scan_front_link"/>
     <child link="laser_frame"/>
-    <origin xyz="${laser_x} 0 ${laser_z}" rpy="0 0 0"/>
+    <origin xyz="0 0 0" rpy="0 0 0"/>
   </joint>
   <!-- ===================================================================== -->
